Commit message: Add SLAM launch file

File: ros2_ws/src/amr_description/urdf/amr_robot.urdf.xacro (robot description, xacro)
@@ -198,5 +198,5 @@
        (= 0.160 + 0.030 = 0.190 m above base_link centre with 320 mm chassis height).
        ===================================================================== -->
-  <link name="laser_frame">
+  <link name="laser">
     <visual>
       <origin xyz="0 0 0" rpy="0 0 0"/>
@@ -223,5 +223,5 @@
   <joint name="laser_joint" type="fixed">
     <parent link="base_link"/>
-    <child  link="laser_frame"/>
+    <child  link="laser"/>
     <origin xyz="0.25 0.0 ${base_height / 2.0 + lidar_height / 2.0}" rpy="0 0 0"/>
   </joint>

Commit message: refactor: reorganize project structure into modules (bringup, description, navigation, hardware) and integrate slam_toolbox

File: ros2_ws/src/amr_description/urdf/amr_robot.urdf.xacro (robot description, xacro)
@@ -3,12 +3,12 @@
   <xacro:include filename="$(find amr_description)/urdf/gazebo_control.xacro"/>
   <!-- =====================================================================
-       Physical hardware dimensions — SLLIDAR C1 + 130 mm drive wheels
+       Physical hardware dimensions — SLLIDAR C1 + 125 mm drive wheels
        ===================================================================== -->
   <xacro:property name="base_length"    value="0.640"/>   <!-- X, front-back -->
   <xacro:property name="base_width"     value="0.540"/>   <!-- Y, side-side  -->
   <xacro:property name="base_height"    value="0.320"/>   <!-- Z             -->
-  <xacro:property name="wheel_radius"   value="0.065"/>
+  <xacro:property name="wheel_radius"   value="0.0625"/>
   <xacro:property name="wheel_width"    value="0.040"/>
-  <xacro:property name="wheel_y"        value="0.270"/>   <!-- |Y| from centre = base_width/2 → 540 mm separation -->
+  <xacro:property name="wheel_y"        value="0.325"/>   <!-- |Y| from centre → 650 mm total track width -->
   <xacro:property name="wheel_x"        value="-0.100"/>  <!-- rear-biased axle position -->
   <xacro:property name="caster_radius"  value="0.025"/>
@@ -60,7 +60,7 @@
         <origin xyz="0 0 0" rpy="0 0 0"/>
         <mass value="1.0"/>
-        <inertia ixx="0.001190" ixy="0" ixz="0"
-                                 iyy="0.002113" iyz="0"
-                                                 izz="0.001190"/>
+        <inertia ixx="0.001110" ixy="0" ixz="0"
+                                 iyy="0.001953" iyz="0"
+                                                 izz="0.001110"/>
       </inertial>
     </link>

Commit message: fix: set robot joints to fixed for stable presentation mode

File: ros2_ws/src/amr_description/urdf/amr_robot.urdf.xacro (robot description, xacro)
@@ -66,9 +66,9 @@
     </link>
     <!-- Wheel centre is at the bottom face of the base (same height as wheel_radius) -->
-    <joint name="${name}_wheel_joint" type="continuous">
+    <!-- PRESENTATION MODE: fixed joint — revert to type="continuous" + axis for live odometry -->
+    <joint name="${name}_wheel_joint" type="fixed">
       <parent link="base_link"/>
       <child  link="${name}_wheel_link"/>
       <origin xyz="${wheel_x} ${y_sign * wheel_y} ${-(base_height / 2.0)}" rpy="0 0 0"/>
-      <axis xyz="0 1 0"/>
     </joint>
   </xacro:macro>
@@ -185,10 +185,9 @@
     </inertial>
   </link>
-  <joint name="lift_joint" type="prismatic">
+  <!-- PRESENTATION MODE: fixed joint — revert to type="prismatic" + axis + limit for live control -->
+  <joint name="lift_joint" type="fixed">
     <parent link="base_link"/>
     <child  link="lift_link"/>
     <origin xyz="0.0 0 ${base_height / 2.0 + lift_height / 2.0}" rpy="0 0 0"/>
-    <axis xyz="0 0 1"/>
-    <limit lower="0.0" upper="0.5" effort="100" velocity="0.1"/>
   </joint>
   <!-- =====================================================================

Commit message: fix the 2700 in ros2

File: ros2_ws/src/amr_description/urdf/amr_robot.urdf.xacro (robot description, xacro)
@@ -113,5 +113,5 @@
     <parent link="base_footprint"/>
     <child  link="base_link"/>
-    <origin xyz="0 0 ${base_z}" rpy="0 0 0"/>
+    <origin xyz="0 0 ${base_z}" rpy="0 0 3.14159"/>
   </joint>
   <!-- =====================================================================
