Commit message: fix: remove 180° yaw rotation from base_footprint_joint
The rpy="0 0 3.14159" was flipping the robot 180° causing it to appear
moving backward in RViz while physically moving forward.

Co-Authored-By: Claude Sonnet 4.6 <noreply@anthropic.com>
Claude-Session: https://claude.ai/code/session_01398Y6ZFw1hy4skUhHrX21f

File: ros2_ws/src/amr_description/urdf/amr_robot.urdf.xacro (robot description, xacro)
@@ -113,5 +113,5 @@
     <parent link="base_footprint"/>
     <child  link="base_link"/>
-    <origin xyz="0 0 ${base_z}" rpy="0 0 3.14159"/>
+    <origin xyz="0 0 ${base_z}" rpy="0 0 0"/>
   </joint>
   <!-- =====================================================================

Commit message: fix: change wheel joints from fixed to continuous for live odometry
Wheels were defined as fixed joints (presentation mode), preventing
ROS from tracking wheel rotation. Now continuous with Y-axis rotation
so encoder odometry and SLAM work correctly on real hardware.

Co-Authored-By: Claude Sonnet 4.6 <noreply@anthropic.com>
Claude-Session: https://claude.ai/code/session_01398Y6ZFw1hy4skUhHrX21f

File: ros2_ws/src/amr_description/urdf/amr_robot.urdf.xacro (robot description, xacro)
@@ -66,9 +66,9 @@
     </link>
     <!-- Wheel centre is at the bottom face of the base (same height as wheel_radius) -->
-    <!-- PRESENTATION MODE: fixed joint — revert to type="continuous" + axis for live odometry -->
-    <joint name="${name}_wheel_joint" type="fixed">
+    <joint name="${name}_wheel_joint" type="continuous">
       <parent link="base_link"/>
       <child  link="${name}_wheel_link"/>
       <origin xyz="${wheel_x} ${y_sign * wheel_y} ${-(base_height / 2.0)}" rpy="0 0 0"/>
+      <axis xyz="0 1 0"/>
     </joint>
   </xacro:macro>

Commit message: fix: move lidar and camera to rear of robot base_link
Relocate laser joint from X=+0.25 to X=-0.25 and camera joint from
X=+0.32 to X=-0.32, rotating camera 180° to face rearward (-X).

Co-Authored-By: Claude Sonnet 4.6 <noreply@anthropic.com>

File: ros2_ws/src/amr_description/urdf/amr_robot.urdf.xacro (robot description, xacro)
@@ -193,5 +193,5 @@
   <!-- =====================================================================
        SLLIDAR C1  (topic: /scan, frame: laser)
-       Front of the top surface: X = +0.25 m from base_link centre.
+       Rear of the top surface: X = -0.25 m from base_link centre.
        Joint Z = base_height/2 + lidar_height/2 → cylinder bottom flush with chassis top
        (= 0.160 + 0.030 = 0.190 m above base_link centre with 320 mm chassis height).
@@ -227,10 +227,10 @@
     <parent link="base_link"/>
     <child  link="laser"/>
-    <origin xyz="0.25 0.0 ${base_height / 2.0 + lidar_height / 2.0}" rpy="0 0 0"/>
+    <origin xyz="-0.25 0.0 ${base_height / 2.0 + lidar_height / 2.0}" rpy="0 0 0"/>
   </joint>
   <!-- =====================================================================
        Orbbec Astra Pro depth camera  (topic: /camera/depth/points)
-       Mounted on the front face of base_link, centred on the chassis height,
-       facing forward (+X). Origin X = 0.32 m = front edge of base_link.
+       Mounted on the rear face of base_link, centred on the chassis height,
+       facing rearward (-X). Origin X = -0.32 m = rear edge of base_link.
        ===================================================================== -->
   <link name="camera_link">
@@ -260,5 +260,5 @@
     <parent link="base_link"/>
     <child  link="camera_link"/>
-    <origin xyz="0.32 0 0" rpy="0 0 0"/>
+    <origin xyz="-0.32 0 0" rpy="0 0 ${pi}"/>
   </joint>
 </robot>

Commit message: fix: flip drive direction so LiDAR side is robot front
- URDF: rotate base_footprint_joint 180 deg around Z so LiDAR appears at +X
- serial_bridge: add flip_drive_direction param; negates linear cmd to Teensy
  and negates measured vx so forward = LiDAR-first throughout the stack
- bringup: enable flip_drive_direction=True for physical robot

This fixes backwards navigation in Nav2 and removes the zig-zag caused
by the 180-degree frame mismatch between URDF and physical robot.

Co-Authored-By: Claude Sonnet 4.6 <noreply@anthropic.com>

File: ros2_ws/src/amr_description/urdf/amr_robot.urdf.xacro (robot description, xacro)
@@ -113,5 +113,5 @@
     <parent link="base_footprint"/>
     <child  link="base_link"/>
-    <origin xyz="0 0 ${base_z}" rpy="0 0 0"/>
+    <origin xyz="0 0 ${base_z}" rpy="0 0 ${pi}"/>
   </joint>
   <!-- =====================================================================

Commit message: fix: correct URDF wheel/caster positions to match physical robot layout
After the 180-degree base_footprint flip, wheel_x must be positive so
drive wheels appear behind centre (toward caster/back side) in RViz.
Rear casters repositioned to x=+0.10 so all 4 casters appear at the
back of the robot in the flipped frame, matching physical hardware.

Co-Authored-By: Claude Sonnet 4.6 <noreply@anthropic.com>

File: ros2_ws/src/amr_description/urdf/amr_robot.urdf.xacro (robot description, xacro)
@@ -11,5 +11,5 @@
   <xacro:property name="wheel_width"    value="0.040"/>
   <xacro:property name="wheel_y"        value="0.325"/>   <!-- |Y| from centre → 650 mm total track width -->
-  <xacro:property name="wheel_x"        value="-0.100"/>  <!-- rear-biased axle position -->
+  <xacro:property name="wheel_x"        value="0.100"/>   <!-- axle 22 cm from rear → appears behind centre after 180° frame flip -->
   <xacro:property name="caster_radius"  value="0.025"/>
   <!-- Scissor-lift platform -->
@@ -153,6 +153,6 @@
   <xacro:caster name="front_left"  x_pos=" 0.260" y_pos=" 0.200"/>
   <xacro:caster name="front_right" x_pos=" 0.260" y_pos="-0.200"/>
-  <xacro:caster name="rear_left"   x_pos="-0.260" y_pos=" 0.200"/>
-  <xacro:caster name="rear_right"  x_pos="-0.260" y_pos="-0.200"/>
+  <xacro:caster name="rear_left"   x_pos=" 0.100" y_pos=" 0.200"/>
+  <xacro:caster name="rear_right"  x_pos=" 0.100" y_pos="-0.200"/>
   <!-- =====================================================================
        Scissor-lift platform
